File: register-module/a-register.sch (KiCad schematic (older format))
At the start: 22 parts

Commit message: Register module complete, add project library folder
Parts:
- C1, C2, C3: renamed from C?; value C -> 100nF
- R1, R2, R3, R4, R5, R6, R7, R8: renamed from R?; value R -> 220
- gave numbers to parts that had none: 11
Connections:
- net A0: now also D8.2 (A), U1.9 (A7), U3.6 (Q3); no longer D1.2 (A), U1.2 (A0), U2.3 (Q0)
- net A1: now also D7.2 (A), U1.8 (A6), U3.5 (Q2); no longer D2.2 (A), U1.3 (A1), U2.4 (Q1)
- net A2: now also D6.2 (A), U1.7 (A5), U3.4 (Q1); no longer D3.2 (A), U1.4 (A2), U2.5 (Q2)
- net A3: now also D5.2 (A), U1.6 (A4), U3.3 (Q0); no longer D4.2 (A), U1.5 (A3), U2.6 (Q3)
- net A4: now also D4.2 (A), U1.5 (A3), U2.6 (Q3); no longer D5.2 (A), U1.6 (A4), U3.3 (Q0)
- net A5: now also D3.2 (A), U1.4 (A2), U2.5 (Q2); no longer D6.2 (A), U1.7 (A5), U3.4 (Q1)
- net A6: now also D2.2 (A), U1.3 (A1), U2.4 (Q1); no longer D7.2 (A), U1.8 (A6), U3.5 (Q2)
- net A7: now also D1.2 (A), U1.2 (A0), U2.3 (Q0); no longer D8.2 (A), U1.9 (A7), U3.6 (Q3)
- net BUS_0 renamed S0
- net BUS_1 renamed S1
- net BUS_2 renamed S2
- net BUS_3 renamed S3
- net BUS_4 renamed S4
- net BUS_5 renamed S5
- net BUS_6 renamed S6
- net BUS_7 renamed S7
- net ~A0 renamed ~AO
Other:
- moved on the sheet: C2, U2
